File: schematic/airquality.kicad_pcb (KiCad board)
At the start: 2 copper layers, 40 x 98 mm, 59 parts, among them J1 Conn_01x08_MountingPin, Q1 BC817, Q2 BC817, U1 ESP32-WROOM-32D, U2 CH340C, U4 BME280, U5 SGP30, U6 PMS5003, U7 SN74LV1T34DCK, U8 AMS1117-3.3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

Commit message: New board revision
Parts:
- removed J1: Conn_01x08_MountingPin, Connector_Molex:Molex_PicoBlade_53261-0871_1x08-1MP_P1.25mm_Horizontal
- removed JP1: SolderJumper_3_Bridged12, Jumper:SolderJumper-3_P1.3mm_Bridged12_RoundedPad1.0x1.5mm
- removed U6: PMS5003, airquality_footprints:PMS5003
- added C23: 1uF, Capacitor_SMD:C_0603_1608Metric, F.Cu at (79.2, 115.2)
- added R13: 4.7, Resistor_SMD:R_0603_1608Metric, F.Cu at (70.2, 114.8)
- added U3: PMS7003T, airquality_footprints:PMS7003, B.Cu at (86.0, 107.3)
- C8: value 100nF -> 1uF
- C9: value 100nF -> 22uF
- U4: value BME280 -> SGP41-D-R4; footprint Package_LGA:Bosch_LGA-8_2.5x2.5mm_P0.65mm_ClockwisePinNumbering -> airquality_footprints:XDCR_SGP41-D-R4
- USB1: moved to B.Cu
- moved C8 59.3 mm to (72.5, 114.8), turned to -90 degrees
- moved U4 55.5 mm to (76.1, 114.7)
- moved C17 40.4 mm to (67.8, 87.8), turned to -90 degrees
- moved U8 35.9 mm to (72.4, 87.2), turned to 90 degrees
- moved C16 30.3 mm to (77.0, 88.0), turned to 90 degrees
- moved R3 29.2 mm to (75.5, 127.2)
- moved R4 29.2 mm to (79.5, 127.2)
- moved R6 29.2 mm to (73.5, 127.2)
- moved R7 29.2 mm to (77.5, 127.2)
- moved C13 17.7 mm to (72.2, 95.8)
- moved C15 16.3 mm to (70.9, 117.9)
- moved C18 16.3 mm to (74.0, 120.7)
- moved C6 16.3 mm to (75.7, 120.7)
- moved U5 16.3 mm to (78.6, 120.6)
- moved U9 16.3 mm to (70.9, 120.6)
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Connections:
- C8 pad 1: +3V3 -> Net-(U4-VDD)
- R11 pad 1: PMS_RESET -> +3V3
- R11 pad 2: GND -> PMS_RESET
- R12 pad 1: +3V3 -> PMS_SET
- R12 pad 2: PMS_SET -> GND
- U4 pad 1: GND -> Net-(U4-VDD)
- U4 pad 2: +3V3 -> GND
- U4 pad 4: SCL -> GND
- U4 pad 5: Net-(JP1-C) -> +3V3
- U4 pad 6: +3V3 -> SCL
Routing:
- net GND: track 20.4 -> 4.78 mm, vias 127 -> 133
- net SDA: track 110.6 -> 124.1 mm, vias 8 -> 6
- net D+: track 22.1 -> 33.4 mm
- net D-: track 22.1 -> 33.4 mm
- net ESP_EN: track 71.7 -> 61.6 mm
- net Net-(JP1-C): track 9.43 -> 0.00 mm
- net PMS_TX: track 51.7 -> 44.8 mm, vias 2 -> 1
- net PMS_RX: track 49.3 -> 44.6 mm, vias 2 -> 1
- net Net-(U4-VDD): track 0.00 -> 4.58 mm
- net VBUS: track 153.6 -> 150.1 mm
- net +3V3: track 199.0 -> 195.9 mm, vias 4 -> 2
- net PMS_RESET: track 57.3 -> 54.5 mm, vias 2 -> 1
- net Net-(USB1-CC1): track 11.1 -> 12.1 mm
- net Net-(USB1-CC2): track 13.4 -> 12.6 mm
- net PMS_SET: track 49.2 -> 49.3 mm, vias 2 -> 1
Other:
- outline, holes or cut-outs redrawn
