File: schematic/airquality.kicad_sch (KiCad schematic)
At the start: 55 parts, among them J1 TYPE-C-31-M-12, Q1 BC817, Q2 BC817, U1 ESP32-WROOM-32D, U2 BME280, U3 SN74LV1T34DCK, U4 SGP30, U5 TLV70218_SOT23-5, U6 PMS7003, U7 AMS1117-3.3, U8 CH340C, U9 SCD30

Commit message: Fix iluminance pin, add caps, add optional double pullups for I2C, cleaup
Parts:
- added C5, C6: 100nF, Capacitor_SMD:C_0201_0603Metric, symbol Device:C
- added R4, R6: 10K, Resistor_SMD:R_0201_0603Metric, symbol Device:R
- SCD30: renamed from U9; value SCD30 -> SCD30 (CO2)
- renumbered C7 to C10, C9 to C11, C10 to C12, C11 to C13, C12 to C14, C13 to C15, C14 to C16, C15 to C17, C16 to C18, C17 to C19, C18 to C20, C19 to C22, C20 to C23, C5 to C7, C6 to C8, C8 to C9, R8 to R10, R9 to R11, R10 to R12, R4 to R2, R5 to R3, R2 to R5, R3 to R7, R6 to R8, R7 to R9, U7 to U6, U8 to U7, U6 to U9
Connections:
- net +3V3: now also C5.1, C6.1, R4.1, R6.1
- net GND: now also C5.2, C6.2
- net Iluminance: now also U1.9 (IO33); no longer U1.11 (IO26)
- net SCD30_RDY: now also U1.8 (IO32); no longer U1.9 (IO33)
- net SCL: now also R6.2
- net SDA: now also R4.2
Other:
- moved on the sheet: C3, C4, R5

Commit message: Lots of fixes
Parts:
- removed C16: 100nF, Capacitor_SMD:C_0201_0603Metric, symbol Device:C
- removed J1: TYPE-C-31-M-12, symbols:HRO_TYPE-C-31-M-12, symbol TYPE-C-31-M-12:TYPE-C-31-M-12
- added USB1: USB_C_Receptacle, airquality_footprints:Hanbo Electronic MC-802YC-H100, symbol usb-c symbol:USB_C_Receptacle
- BOOT1, RESET1: footprint symbols:GT-TC029B-H025-L1N -> airquality_footprints:GT-TC029B-H025-L1N
- C1, C10, C11, C13, C15, C2, C3, C4, C5, C6, C7, C8, C9: footprint Capacitor_SMD:C_0201_0603Metric -> Capacitor_SMD:C_0603_1608Metric
- C12: renamed from C14; footprint Capacitor_SMD:C_0201_0603Metric -> Capacitor_SMD:C_0603_1608Metric
- C14: renamed from C12; footprint Capacitor_SMD:C_0201_0603Metric -> Capacitor_SMD:C_0603_1608Metric
- C16: renamed from C17; footprint Capacitor_SMD:C_0201_0603Metric -> Capacitor_SMD:C_0603_1608Metric
- C17: renamed from C18; footprint Capacitor_SMD:C_0201_0603Metric -> Capacitor_SMD:C_0603_1608Metric
- C19: renamed from C20; footprint Capacitor_SMD:C_0201_0603Metric -> Capacitor_SMD:C_0603_1608Metric
- C20: renamed from C21; footprint Capacitor_SMD:C_0201_0603Metric -> Capacitor_SMD:C_0603_1608Metric
- C21: renamed from C22; footprint Capacitor_SMD:C_0201_0603Metric -> Capacitor_SMD:C_0603_1608Metric
- C22: renamed from C23; footprint Capacitor_SMD:C_0201_0603Metric -> Capacitor_SMD:C_0603_1608Metric
- D1: footprint LED_THT:LED_D5.0mm_Horizontal_O6.35mm_Z15.0mm -> airquality_footprints:ALS-PDIC243-3B
- R1, R10, R12, R4, R5, R6, R7, R8, R9: footprint Resistor_SMD:R_0201_0603Metric -> Resistor_SMD:R_0603_1608Metric
- R11: footprint Resistor_SMD:R_0201_0603Metric -> Resistor_SMD:R_0603_1608Metric; LCSC (none) -> https://www.lcsc.com/product-detail/Chip-Resistor-Surface-M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
- R2: renamed from R3; footprint Resistor_SMD:R_0201_0603Metric -> Resistor_SMD:R_0603_1608Metric
- R3: renamed from R2; footprint Resistor_SMD:R_0201_0603Metric -> Resistor_SMD:R_0603_1608Metric
- SCD1: renamed from SCD30; footprint symbols:MODULE_SCD30 -> airquality_footprints:MODULE_SCD30
- U1: footprint RF_Module:ESP32-WROOM-32D -> airquality_footprints:ESP32-WROOM-32D
- U4: footprint symbols:SGP30 -> airquality_footprints:SGP30
- U5: symbol Regulator_Linear:TLV70218_SOT23-5 -> tlv70218_sot23-5:TLV70218_SOT23-5
- U8: renamed from U9; footprint symbols:PMS7003 -> airquality_footprints:PMS7003
- renumbered C19 to C18
Connections:
- net D+: now also USB1.A6 (D+), USB1.B6 (D+)
- net D-: now also USB1.A7 (D-), USB1.B7 (D-)
- net GND: now also U5.4 (NC), USB1.A1 (GND), USB1.A12 (GND), USB1.B1 (GND), USB1.B12 (GND), USB1.S1 (SHIELD)
- net VBUS: now also USB1.A4 (VBUS), USB1.A9 (VBUS), USB1.B4 (VBUS), USB1.B9 (VBUS)
- net at R12.1: now also USB1.B5 (CC2)
- net at R11.1: now also USB1.A5 (CC1)
- no-connect marks 29 -> 27
Other:
- moved on the sheet: C21

Commit message: swap PMS7003 with PMS5003
Parts:
- added J1: Conn_01x08_MountingPin, Connector_Molex:Molex_PicoBlade_53261-0871_1x08-1MP_P1.25mm_Horizontal, symbol Connector_Generic_MountingPin:Conn_01x08_MountingPin
- added U6: PMS5003, airquality_footprints:PMS5003, symbol Connector:Conn_01x08_Pin
- renumbered C4 to C1, C15 to C10, C8 to C11, C10 to C12, C18 to C13, C20 to C14, C12 to C15, C19 to C16, C22 to C17, C13 to C18, C7 to C19, C3 to C2, C9 to C20, C17 to C21, C11 to C22, C5 to C3, C6 to C4, C21 to C5, C14 to C6, C1 to C7, C2 to C8, C16 to C9, Q2 to Q1, Q1 to Q2, R11 to R1, R9 to R10, R2 to R11, R3 to R12, R12 to R2, R5 to R3, R7 to R4, R1 to R5, R4 to R6, R6 to R7, R10 to R8, R8 to R9, U7 to U2, U8 to U3, U2 to U4, U4 to U5, U3 to U7, U6 to U8, U5 to U9
Connections:
- net +3V3: no longer R11.1
- net GND: now also R11.2, J1.7 (Pin_7), J1.MP (MountPin), U6.2 (Pin_2)
- net PMS_RESET: now also R11.1, J1.3 (Pin_3), U6.6 (Pin_6); no longer R11.2
- net PMS_RX: now also J1.5 (Pin_5), U6.4 (Pin_4)
- net PMS_SET: now also J1.6 (Pin_6), U6.3 (Pin_3)
- net PMS_TX: now also J1.4 (Pin_4), U6.5 (Pin_5)
- net VBUS: now also J1.8 (Pin_8), U6.1 (Pin_1)
- new net: J1.2 (Pin_2), U6.7 (Pin_7)
- new net: J1.1 (Pin_1), U6.8 (Pin_8)
- no-connect marks 27 -> 29
Other:
- note added: "Particulate sensor - PMS5003"
- note added: "Particulate sensor - PMS7003"
- note removed: "Particulate sensor"
- moved on the sheet: R11

Commit message: New board revision
Parts:
- removed JP1: SolderJumper_3_Bridged12, Jumper:SolderJumper-3_P1.3mm_Bridged12_RoundedPad1.0x1.5mm, symbol Jumper:SolderJumper_3_Bridged12
- removed U4: BME280, Package_LGA:Bosch_LGA-8_2.5x2.5mm_P0.65mm_ClockwisePinNumbering, symbol Sensor:BME280
- added C23: 1uF, Capacitor_SMD:C_0603_1608Metric, symbol Device:C
- added R13: 4.7, Resistor_SMD:R_0603_1608Metric, symbol Device:R
- added U4: SGP41-D-R4, airquality_footprints:XDCR_SGP41-D-R4, symbol sgp41:SGP41-D-R4
- C8: value 100nF -> 1uF; LCSC (none) -> https://www.lcsc.com/product-detail/Multilayer-Ceramic-Capa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
- C9: value 100nF -> 22uF
- J1, U6: now not fitted; now left out of the parts list
- U3: value PMS7003 -> PMS7003T
Connections:
- net +3V3: now also R11.1, C23.1, R13.1, U4.5 (VDDH); no longer C8.1, R12.1
- net GND: now also R12.2, C23.2, U4.2 (VSS), U4.4 (N/A), U4.7 (EXP); no longer R11.2
- net PMS_RESET: now also R11.2; no longer R11.1
- net PMS_SET: now also R12.1; no longer R12.2
- net SCL: now also U4.6 (SCL)
- net SDA: now also U4.3 (SDA)
- new net: C8.1, R13.2, U4.1 (VDD)
Other:
- note added: "Particulate sensor - PMS7003T"
- note added: "SGP41 - VOC and NOx sensor"
- note removed: "Particulate sensor - PMS7003"
- note removed: "Temperature/humidity/pressure"
- moved on the sheet: C7, D1, D3, D4, D5, D6, R11, R12, R5
